File: PCB/BarometricPressureSensor.kicad_pcb (KiCad board)
At the start: 2 copper layers, 104.1 x 67.1 mm, 44 parts, among them J1 USB4105-GF-A, J10 B2B-PH-K-S, J2 54-00125, J4 GTFP08441BEU, J5 2337019-1, J8 B6B-PH-K-S, J9 B3B-PH-K-S, U1 ESP32-S3-DEVKITC-1-N16R8V, U2 DPS368XTSA1, U3 BQ24074RGT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

Commit message: Annotated main board schematic, corrected switch short on main PCB
Routing:
- net +BATT: track 75.2 -> 71.7 mm
